Commit message: se agregaron modelos mejores y estacionamiento

File: src/visualizacion/urdf/dron.urdf (robot description, URDF)
Before this commit: robot dron, 4 links, 3 joints
Links:
- added link propela_1, mass 0.1; collision box size=0.1 0.1 0.1; visual mesh filename=package://visualizacion/models/propela/meshes/propela.obj scale=2 2 2
- added link propela_2, mass 0.1; collision box size=0.1 0.1 0.1; visual mesh filename=package://visualizacion/models/propela/meshes/propela.obj scale=2 2 2
- added link propela_3, mass 0.1; collision box size=0.1 0.1 0.1; visual mesh filename=package://visualizacion/models/propela/meshes/propela.obj scale=2 2 2
- added link propela_4, mass 0.1; collision box size=0.1 0.1 0.1; visual mesh filename=package://visualizacion/models/propela/meshes/propela.obj scale=2 2 2
- link dron_link: geometry collision box size=0.1 0.1 0.1; visual mesh filename=package://visualizacion/models/dron/meshes/djimini4pro.obj scale=2 2 2
Joints:
- added joint dron_to_propela1: type continuous, parent dron_link, child propela_1, origin xyz=0 -0.067 -0.003 rpy=0 0 0, axis 0 0 1
- added joint dron_to_propela2: type continuous, parent dron_link, child propela_2, origin xyz=-0.31 -0.067 -0.003 rpy=0 0 0, axis 0 0 1
- added joint dron_to_propela3: type continuous, parent dron_link, child propela_3, origin xyz=0 0.248 -0.04 rpy=0 0 0, axis 0 0 1
- added joint dron_to_propela4: type continuous, parent dron_link, child propela_4, origin xyz=-0.31 0.248 -0.04 rpy=0 0 0, axis 0 0 1
- joint world_fixed: origin xyz=0 0 0 rpy=0 0 0 -> xyz=0 0 0.22 rpy=0 0 0

Commit message: Ya se puede mover el dron

File: src/visualizacion/urdf/dron.urdf (robot description, URDF)
Before this commit: robot dron, 8 links, 7 joints
Links:
- removed link world_link
- link base_link: mass 5.0 -> None
- link propela_1: mass 0.1 -> 0.01
- link propela_2: mass 0.1 -> 0.01
- link propela_3: mass 0.1 -> 0.01
- link propela_4: mass 0.1 -> 0.01
Joints:
- removed joint world_fixed
- joint dron_to_propela1: origin xyz=0 -0.067 -0.003 rpy=0 0 0 -> xyz=0.155 -0.135 0 rpy=0 0 0
- joint dron_to_propela2: origin xyz=-0.31 -0.067 -0.003 rpy=0 0 0 -> xyz=-0.155 0.135 0 rpy=0 0 0
- joint dron_to_propela3: origin xyz=0 0.248 -0.04 rpy=0 0 0 -> xyz=0.155 0.135 0 rpy=0 0 0
- joint dron_to_propela4: origin xyz=-0.31 0.248 -0.04 rpy=0 0 0 -> xyz=-0.155 -0.135 0 rpy=0 0 0
